File: pcb/snailbot.kicad_pcb (KiCad board)
At the start: 2 copper layers, 64 x 100 mm, 53 parts, among them J1 USB_B_Micro, J2 Conn_01x04_Female, J3 Conn_01x05_Male, J4 Conn_01x06_Female, J5 Conn_01x05_Male, SW1 SW_Push, SW2 SW_Push, SW3 SW_Push, U1 MCP73831-2-OT, U2 MCP1642B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

Commit message: Fixed issues found in prototype
Parts:
- removed G***: LOGO, mc_logo:acasta_s4
- removed NT1: Net-Tie_2, NetTie:NetTie-2_SMD_Pad0.5mm
- removed R16: 100, Resistor_SMD:R_0805_2012Metric_Pad1.15x1.40mm_HandSolder
- added C3: 10n, Capacitor_SMD:C_0805_2012Metric_Pad1.15x1.40mm_HandSolder, F.Cu at (84.0, 42.0)
- added Q1: BSS138, Package_TO_SOT_SMD:SOT-23, F.Cu at (55.5, 40.0)
- R3: value 750k 1% -> 470k 1%
- R4: value 1k -> 470
Connections:
- SW1 pad 1: Net-(R16-Pad1) -> +BATT
- U4 pad 23: Net-(NT1-Pad1) -> PC0
Routing:
- net Net-(NT1-Pad1): track 63.4 -> 0.00 mm, vias 2 -> 0
- net PC0: track 0.00 -> 59.7 mm, vias 0 -> 2
- net +BATT: track 62.0 -> 84.9 mm, vias 0 -> 2
- net Net-(R16-Pad1): track 17.0 -> 0.00 mm, vias 2 -> 0
- net VCC: track 272.5 -> 285.3 mm, vias 1 -> 2
- net PC4: track 90.7 -> 92.4 mm
Other:
- board text added: "2021-08-23"
- board text added: "rev. 3"
- board text added: "snailbot"
- board text removed: "2019-09-21"
- board text removed: "il"
- board text removed: "rev. 2"
- board text removed: "sn"

Commit message: Updated schematics and production files
Parts:
- moved Q1 0.50 mm to (56.0, 40.0)
Routing:
- net VCC: track 285.3 -> 285.8 mm
- net PC0: track 59.7 -> 59.2 mm
Changed lines of the file:
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@@
     (thickness 1.6)
     (drawings 29)
-    (tracks 380)
+    (tracks 378)
     (zones 0)
     (modules 52)
@@
   )
   (module Package_TO_SOT_SMD:SOT-23 (layer F.Cu)
-    (at 55.5 40 90)
+    (at 56 40 90)
     (descr "SOT-23, Standard")
     (tags SOT-23)
@@
   (segment (start 51 42) (end 53 40) (width 0.7) (layer F.Cu) (net 4) (status 10))
   (segment (start 51 42) (end 46.5 42) (width 0.7) (layer F.Cu) (net 4) (status 10))
+  (segment (start 51 23) (end 50 22) (width 0.25) (layer F.Cu) (net 4))
+  (segment (start 50 22) (end 49.1 22) (width 0.25) (layer F.Cu) (net 4) (status 20))
+  (via (at 51 23) (size 0.8) (drill 0.4) (layers F.Cu B.Cu) (net 4))
+  (segment (start 51 23) (end 51 31) (width 0.25) (layer B.Cu) (net 4))
+  (segment (start 54.5 34.5) (end 51 31) (width 0.25) (layer B.Cu) (net 4))
+  (segment (start 54.5 34.225) (end 52.775 32.5) (width 0.25) (layer F.Cu) (net 4))
+  (segment (start 54.5 34.5) (end 54.5 34.225) (width 0.25) (layer F.Cu) (net 4))
+  (via (at 54.5 34.5) (size 0.8) (drill 0.4) (layers F.Cu B.Cu) (net 4))
+  (segment (start 54.5 34.5) (end 56 36) (width 0.25) (layer F.Cu) (net 4))
+  (segment (start 56 36) (end 56 39) (width 0.25) (layer F.Cu) (net 4))
   (segment (start 89.76 60.5) (end 90 60.74) (width 0.4) (layer B.Cu) (net 5) (status 30))
   (segment (start 87.5 60.5) (end 89.76 60.5) (width 0.4) (layer B.Cu) (net 5) (status 30))
@@
   (segment (start 65.88 107) (end 65.88 108.12) (width 0.4) (layer F.Cu) (net 5) (status 10))
   (segment (start 62 112) (end 51.5 112) (width 0.4) (layer F.Cu) (net 5))
+  (segment (start 43.5 43) (end 43.5 58) (width 0.4) (layer B.Cu) (net 5))
+  (segment (start 43.5 30) (end 43.5 43) (width 0.4) (layer B.Cu) (net 5))
+  (via (at 54 43) (size 1) (drill 0.4) (layers F.Cu B.Cu) (net 5))
+  (segment (start 43.5 43) (end 54 43) (width 0.4) (layer B.Cu) (net 5))
+  (segment (start 54 43) (end 54.5 43) (width 0.4) (layer F.Cu) (net 5))
+  (segment (start 55.05 42.45) (end 55.05 41) (width 0.4) (layer F.Cu) (net 5))
+  (segment (start 54.5 43) (end 55.05 42.45) (width 0.4) (layer F.Cu) (net 5))
   (segment (start 82.95 31.5) (end 82.95 34) (width 0.25) (layer F.Cu) (net 6) (status 30))
   (segment (start 82.95 34) (end 82.95 36.5) (width 0.25) (layer F.Cu) (net 6) (status 30))
@@
   (segment (start 85 40) (end 84.5 40.5) (width 0.25) (layer F.Cu) (net 34))
   (segment (start 84.5 40.5) (end 73 40.5) (width 0.25) (layer F.Cu) (net 34))
+  (segment (start 85 41) (end 84.5 40.5) (width 0.25) (layer F.Cu) (net 34))
+  (segment (start 85 42) (end 85 41) (width 0.25) (layer F.Cu) (net 34))
   (segment (start 86.42 50.58) (end 90 50.58) (width 0.25) (layer F.Cu) (net 35) (status 20))
   (segment (start 83.5 53.5) (end 86.42 50.58) (width 0.25) (layer F.Cu) (net 35))
@@
   (segment (start 94.5 44.5) (end 94.5 56.5) (width 0.25) (layer F.Cu) (net 47))
   (segment (start 93 43) (end 93.5 43.5) (width 0.25) (layer B.Cu) (net 47))
-  (segment (start 51 23) (end 50 22) (width 0.25) (layer F.Cu) (net 4))
-  (segment (start 50 22) (end 49.1 22) (width 0.25) (layer F.Cu) (net 4) (status 20))
-  (via (at 51 23) (size 0.8) (drill 0.4) (layers F.Cu B.Cu) (net 4))
-  (segment (start 51 23) (end 51 31) (width 0.25) (layer B.Cu) (net 4))
-  (segment (start 55.05 36) (end 55.05 35.05) (width 0.25) (layer F.Cu) (net 4) (status 10))
-  (via (at 54.5 34.5) (size 0.8) (drill 0.4) (layers F.Cu B.Cu) (net 4))
-  (segment (start 55.05 35.05) (end 54.5 34.5) (width 0.25) (layer F.Cu) (net 4))
-  (segment (start 54.5 34.5) (end 51 31) (width 0.25) (layer B.Cu) (net 4))
-  (segment (start 55.05 38.55) (end 55.5 39) (width 0.25) (layer F.Cu) (net 4))
-  (segment (start 55.05 36) (end 55.05 38.55) (width 0.25) (layer F.Cu) (net 4))
-  (segment (start 54.5 34.225) (end 52.775 32.5) (width 0.25) (layer F.Cu) (net 4))
-  (segment (start 54.5 34.5) (end 54.5 34.225) (width 0.25) (layer F.Cu) (net 4))
-  (segment (start 43.5 43) (end 53 43) (width 0.4) (layer B.Cu) (net 5))
-  (via (at 53 43) (size 1) (drill 0.4) (layers F.Cu B.Cu) (net 5))
-  (segment (start 43.5 43) (end 43.5 58) (width 0.4) (layer B.Cu) (net 5))
-  (segment (start 43.5 30) (end 43.5 43) (width 0.4) (layer B.Cu) (net 5))
-  (segment (start 53 43) (end 54 43) (width 0.4) (layer F.Cu) (net 5))
-  (segment (start 54.55 42.45) (end 54.55 41) (width 0.4) (layer F.Cu) (net 5))
-  (segment (start 54 43) (end 54.55 42.45) (width 0.4) (layer F.Cu) (net 5))
-  (segment (start 85 41) (end 84.5 40.5) (width 0.25) (layer F.Cu) (net 34))
-  (segment (start 85 42) (end 85 41) (width 0.25) (layer F.Cu) (net 34))
+  (segment (start 92 42) (end 93.5 43.5) (width 0.25) (layer B.Cu) (net 47))
+  (segment (start 75.5 42) (end 92 42) (width 0.25) (layer B.Cu) (net 47))
   (segment (start 73 44.5) (end 75.5 42) (width 0.25) (layer B.Cu) (net 47))
-  (segment (start 75.5 42) (end 92 42) (width 0.25) (layer B.Cu) (net 47))
-  (segment (start 92 42) (end 93.5 43.5) (width 0.25) (layer B.Cu) (net 47))
-  (via (at 56.5 43) (size 0.8) (drill 0.4) (layers F.Cu B.Cu) (net 47))
-  (segment (start 73 44.5) (end 58 44.5) (width 0.25) (layer B.Cu) (net 47))
-  (segment (start 58 44.5) (end 56.5 43) (width 0.25) (layer B.Cu) (net 47))
-  (segment (start 56.45 42.95) (end 56.45 41) (width 0.25) (layer F.Cu) (net 47))
-  (segment (start 56.5 43) (end 56.45 42.95) (width 0.25) (layer F.Cu) (net 47))
+  (via (at 57 43) (size 0.8) (drill 0.4) (layers F.Cu B.Cu) (net 47))
+  (segment (start 73 44.5) (end 58.5 44.5) (width 0.25) (layer B.Cu) (net 47))
+  (segment (start 58.5 44.5) (end 57 43) (width 0.25) (layer B.Cu) (net 47))
+  (segment (start 56.95 42.95) (end 56.95 41) (width 0.25) (layer F.Cu) (net 47))
+  (segment (start 57 43) (end 56.95 42.95) (width 0.25) (layer F.Cu) (net 47))
   (zone (net 2) (net_name GND) (layer F.Cu) (hatch edge 0.508)
     (connect_pads (clearance 0.5))
